File: rgb2vga_deltas.kicad_pcb (KiCad board)
At the start: 2 copper layers, 63.3 x 81.6 mm, 35 parts, among them J1 DE15_Receptacle_HighDensity, J2 Conn_01x09, Q1 BC547, Q2 BC547, Q3 BC547, Q4 BC547, Q5 BC547, Q6 BC547, Q7 BC547, U1 Pico

Commit message: Board routed
Parts:
- moved J2 1.06 mm to (65.8, 127.1)
Routing:
- net GND: track 205.2 -> 0.00 mm
- net Net-(J1-Pad1): track 21.5 -> 28.7 mm
- net +5V: track 49.0 -> 53.2 mm
- net GP1: track 46.0 -> 48.9 mm
- net Net-(J1-Pad14): track 21.7 -> 24.4 mm
- net Net-(J1-Pad13): track 16.8 -> 19.1 mm
- net GP6: track 53.1 -> 55.3 mm
- net GP3: track 47.3 -> 49.0 mm
- net G: track 13.0 -> 11.4 mm
- net F: track 13.6 -> 14.7 mm
- net GP2: track 45.7 -> 46.7 mm
- net R: track 10.8 -> 9.85 mm
- net Net-(J1-Pad2): track 10.7 -> 11.5 mm
- net GP4: track 49.0 -> 49.8 mm
- net B: track 16.2 -> 15.5 mm
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- added copper zone on B.Cu, net GND
- added copper zone on F.Cu, net GND
