File: rgb2vga_deltas.kicad_sch (KiCad schematic)
At the start: 7 parts, among them J1 DE15_Receptacle_HighDensity

Commit message: Update rgb2vga_deltas.kicad_sch
Parts:
- added U1: Pico, rgb2bga_test:RPi_Pico_SMD_TH, symbol rgb2vga_test:Pico
Changed lines of the file:
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@@
+    )
+  )
+  (symbol (lib_id "rgb2vga_test:Pico") (at 72.39 117.475 0) (unit 1)
+    (in_bom yes) (on_board yes) (dnp no) (fields_autoplaced)
+    (property "Reference" "U1" (at 72.39 86.36 0)
+      (effects (font (size 1.27 1.27)))
+    )
+    (property "Value" "Pico" (at 72.39 88.9 0)
+      (effects (font (size 1.27 1.27)))
+    )
+    (property "Footprint" "rgb2bga_test:RPi_Pico_SMD_TH" (at 72.39 117.475 90)
+      (effects (font (size 1.27 1.27)) hide)
+    )
+    (property "Datasheet" "" (at 72.39 117.475 0)
+      (effects (font (size 1.27 1.27)) hide)
+    )
+    (pin "30")
+    (pin "34")
+    (pin "35")
+    (pin "5")
+    (pin "7")
+    (pin "27")
+    (pin "2")
+    (pin "25")
+    (pin "12")
+    (pin "21")
+    (pin "31")
+    (pin "23")
+    (pin "29")
+    (pin "38")
+    (pin "11")
+    (pin "42")
+    (pin "13")
+    (pin "6")
+    (pin "10")
+    (pin "15")
+    (pin "17")
+    (pin "40")
+    (pin "8")
+    (pin "9")
+    (pin "1")
+    (pin "22")
+    (pin "24")
+    (pin "16")
+    (pin "19")
+    (pin "26")
+    (pin "3")
+    (pin "33")
+    (pin "32")
+    (pin "39")
+    (pin "41")
+    (pin "43")
+    (pin "37")
+    (pin "4")
+    (pin "36")
+    (pin "14")
+    (pin "18")
+    (pin "20")
+    (pin "28")
+    (instances
+      (project "rgb2vga_deltas"
+        (path "/1e94bb5d-73d6-4764-bb5c-d48b64a032b6"
+          (reference "U1") (unit 1)
+        )
+      )
     )
   )

Commit message: First version release
Parts:
- added C1, C2, C3: 0,1uF, Capacitor_THT:C_Disc_D7.0mm_W2.5mm_P5.00mm, symbol Device:C
- added J2: Conn_01x09, Connector_PinHeader_2.54mm:PinHeader_1x09_P2.54mm_Vertical, symbol Connector_Generic:Conn_01x09
- added Q1, Q2, Q3, Q4, Q5, Q6, Q7: BC547, Package_TO_SOT_THT:TO-92_Inline, symbol Transistor_BJT:BC547
- added R10, R11, R12, R13, R14, R15, R16, R17, R18, R19, R20, R21, R22, R9: 1K, Resistor_THT:R_Axial_DIN0207_L6.3mm_D2.5mm_P10.16mm_Horizontal, symbol Device:R
- added R7, R8: 100R, Resistor_THT:R_Axial_DIN0207_L6.3mm_D2.5mm_P10.16mm_Horizontal, symbol Device:R
- J1: footprint (none) -> Connector_Dsub:DSUB-15-HD_Female_Horizontal_P2.29x1.98mm_EdgePinOffset3.03mm_Housed_MountingHolesOffset4.94mm
- R1, R2, R3, R4, R5, R6: footprint (none) -> Resistor_THT:R_Axial_DIN0207_L6.3mm_D2.5mm_P10.16mm_Horizontal
Connections:
- net GP10: now reaches R3.1
- net GP10: now also U1.14 (GPIO10)
- net GP8: now reaches R1.1
- net GP8: now also U1.11 (GPIO8)
- net GP12: now reaches R5.1
- net GP12: now also U1.16 (GPIO12)
- net GP13: now reaches R6.1
- net GP13: now also U1.17 (GPIO13)
- net GND: now reaches J1.10
- net GND: now also J1.5, J1.6, J1.7, J1.8, U1.13 (GND), U1.18 (GND), U1.23 (GND), U1.28 (GND), U1.3 (GND), U1.33 (AGND), U1.38 (GND), U1.8 (GND), C1.2, C2.2, C3.2, J2.9 (Pin_9)
- net at J1.13: now also R7.1
- net at J1.14: now also R8.1
- net GP11: now reaches R4.1
- net GP11: now also U1.15 (GPIO11)
- net GP9: now reaches R2.1
- net GP9: now also U1.12 (GPIO9)
- net GP0: now reaches U1.1 (GPIO0)
- net GP0: now also Q7.1 (C), R22.1
- net GP14: now reaches U1.19 (GPIO14)
- net GP14: now also R7.2
- net GP1: now reaches U1.2 (GPIO1)
- net GP1: now also Q6.1 (C), R20.1
- net GP15: now reaches U1.20 (GPIO15)
- net GP15: now also R8.2
- net +3.3V: now reaches U1.36 (3V3)
- net +3.3V: now also C1.1, C2.1, R10.2, R11.2, R12.2, R13.2, R14.2, R15.2, R16.2, R17.2, R18.2, R19.2, R20.2, R21.2, R22.2, R9.2
- net GP2: now reaches U1.4 (GPIO2)
- net GP2: now also Q5.1 (C), R18.1
- net +5V: now reaches U1.40 (VBUS)
- net +5V: now also C3.1, J2.8 (Pin_8)
- net GP3: now reaches U1.5 (GPIO3)
- net GP3: now also Q4.1 (C), R16.1
- net GP4: now reaches U1.6 (GPIO4)
- net GP4: now also Q3.1 (C), R14.1
- net GP5: now reaches U1.7 (GPIO5)
- net GP5: now also Q2.1 (C), R12.1
- net GP6: now reaches U1.9 (GPIO6)
- net GP6: now also Q1.1 (C), R10.1
- new net: Q3.2 (B), R13.1
- new net: Q5.2 (B), R17.1
- new net: Q7.2 (B), R21.1
- new net: Q1.2 (B), R9.1
- new net: Q2.2 (B), R11.1
- new net: Q4.2 (B), R15.1
- new net: Q6.2 (B), R19.1
- new net B: J2.7 (Pin_7), Q7.3 (E)
- new net F: J2.1 (Pin_1), Q1.3 (E)
- new net G: J2.6 (Pin_6), Q6.3 (E)
- new net I: J2.4 (Pin_4), Q4.3 (E)
- new net KSI: J2.2 (Pin_2), Q2.3 (E)
- new net R: J2.5 (Pin_5), Q5.3 (E)
- new net SSI: J2.3 (Pin_3), Q3.3 (E)
- no-connect marks 0 -> 23
Other:
- moved on the sheet: R2, R3, R5, U1
